Commit message: Updated RRR code with PD control and a maybe working safety filter

File: RRR_manipulator_description/RRR_mobile.urdf (robot description, URDF)
Before this commit: robot onshape, 6 links, 5 joints
Links:
- added link prismatic_x
- added link prismatic_y
Joints:
- removed joint world2base
- added joint px2py: type prismatic, parent prismatic_x, child prismatic_y, origin xyz=0 0 0 rpy=0 0 0, axis 1 0 0, limit effort=1 velocity=20
- added joint py2base: type prismatic, parent prismatic_y, child linkBase, origin xyz=0 0 0 rpy=0 0 1.57079632679, axis 1 0 0, limit effort=1 velocity=20
- added joint world2px: type fixed, parent world, child prismatic_x, origin xyz=0 -0.01750000 0 rpy=0 0 0
